Commit message: add: wheels and sensors to robot xacro file

File: src/a1_bot/urdf/a1_bot.xacro (robot description, xacro)
@@ -3,5 +3,5 @@
   <link name="robot_footprint"></link>
   <joint name="robot_footprint_joint" type="fixed">
-    <origin xyz="0 0 0.099" rpy="0 0 0" /> <!-- keep robot wheels on the groud (offset value as per robot visual)-->
+    <origin xyz="0 0 0.124" rpy="0 0 0" /> <!-- keep robot wheels on the groud (offset value as per robot visual)-->
     <parent link="robot_footprint"/>
     <child link="chassis" />
@@ -31,5 +31,5 @@
     </visual>
     <collision name='back_caster_collision'>
-      <origin xyz="-0.15 0 -0.05" rpy=" 0 0 0"/>
+      <origin xyz="-0.15 0 -0.075" rpy=" 0 0 0"/>
       <geometry>
         <sphere radius="0.0499"/>
@@ -37,5 +37,5 @@
     </collision>
     <visual name='back_caster_visual'>
-      <origin xyz="-0.15 0 -0.05" rpy=" 0 0 0"/>
+      <origin xyz="-0.15 0 -0.075" rpy=" 0 0 0"/>
       <geometry>
         <sphere radius="0.05"/>
@@ -43,5 +43,5 @@
     </visual>
     <collision name='front_caster_collision'>
-      <origin xyz="0.15 0 -0.05" rpy=" 0 0 0"/>
+      <origin xyz="0.15 0 -0.075" rpy=" 0 0 0"/>
       <geometry>
         <sphere radius="0.0499"/>
@@ -49,5 +49,5 @@
     </collision>
     <visual name='front_caster_visual'>
-      <origin xyz="0.15 0 -0.05" rpy=" 0 0 0"/>
+      <origin xyz="0.15 0 -0.075" rpy=" 0 0 0"/>
       <geometry>
         <sphere radius="0.05"/>
@@ -55,3 +55,131 @@
     </visual>
   </link>
+  <gazebo reference="chassis">
+     <material>Gazebo/Orange</material>
+  </gazebo>
+  <gazebo reference="left_wheel">
+     <material>Gazebo/Blue</material>
+  </gazebo>
+  <gazebo reference="right_wheel">
+     <material>Gazebo/Blue</material>
+  </gazebo>
+  <gazebo reference="camera">
+     <material>Gazebo/Red</material>
+  </gazebo>
+  <link name="left_wheel">
+    <inertial>
+       <origin xyz="0 0 0" rpy="0 1.5707 1.5707"/>
+       <mass value="5"/>
+       <inertia ixx="0.1" ixy="0" ixz="0" iyy="0.1" iyz="0" izz="0.1"/>
+     </inertial>
+    <visual>
+      <origin xyz="0 0 0" rpy="0 1.5707 1.5707"/>
+      <geometry>
+        <cylinder length="0.05" radius="0.05"/>
+      </geometry>
+    </visual>
+    <collision>
+      <origin xyz="0 0 0" rpy="0 1.5707 1.5707"/>
+      <geometry>
+        <cylinder length="0.05" radius="0.05"/>
+      </geometry>
+    </collision>
+  </link>
+  <joint type="continuous" name="left_wheel_hinge">
+    <origin xyz="0 0.15 -0.075" rpy="0 0 0"/>
+    <child link="left_wheel"/>
+    <parent link="chassis"/>
+    <axis xyz="0 1 0" rpy="0 0 0"/>
+    <limit effort="10000" velocity="1000"/>
+    <dynamics damping="1.0" friction="1.0"/>
+  </joint>
+  <link name="right_wheel">
+    <inertial>
+       <origin xyz="0 0 0" rpy="0 1.5707 1.5707"/>
+       <mass value="5"/>
+       <inertia ixx="0.1" ixy="0" ixz="0" iyy="0.1" iyz="0" izz="0.1"/>
+     </inertial>
+    <visual>
+      <origin xyz="0 0 0" rpy="0 1.5707 1.5707"/>
+      <geometry>
+        <cylinder length="0.05" radius="0.05"/>
+      </geometry>
+    </visual>
+    <collision>
+      <origin xyz="0 0 0" rpy="0 1.5707 1.5707"/>
+      <geometry>
+        <cylinder length="0.05" radius="0.05"/>
+      </geometry>
+    </collision>
+  </link>
+  <joint type="continuous" name="right_wheel_hinge">
+    <origin xyz="0 -0.15 -0.075" rpy="0 0 0"/>
+    <child link="right_wheel"/>
+    <parent link="chassis"/>
+    <axis xyz="0 1 0" rpy="0 0 0"/>
+    <limit effort="10000" velocity="1000"/>
+    <dynamics damping="1.0" friction="1.0"/>
+  </joint>
+  <link name="camera">
+    <origin xyz="0 0 0" rpy="0 0 0"/>
+    <inertial>
+       <origin xyz="0 0 0" rpy="0 0 0"/>
+       <mass value="0.1"/>
+       <inertia ixx="1e-6" ixy="0" ixz="0" iyy="1e-6" iyz="0" izz="1e-6"/>
+     </inertial>
+    <visual>
+      <origin xyz="0 0 0" rpy="0 0 0"/>
+      <geometry>
+        <box size="0.05 0.05 0.05"/>
+      </geometry>
+    </visual>
+    <collision>
+      <origin xyz="0 0 0" rpy="0 0 0"/>
+      <geometry>
+        <box size="0.05 0.05 0.05"/>
+      </geometry>
+    </collision>
+  </link>
+  <joint type="fixed" name="camera_joint">
+    <origin xyz="0.225 0 0" rpy="0 0 0"/>
+    <child link="camera"/>
+    <parent link="chassis"/>
+    <axis xyz="0 1 0" rpy="0 0 0"/>
+    <limit effort="10000" velocity="1000"/>
+    <dynamics damping="1.0" friction="1.0"/>
+  </joint>
+  <link name="hokuyo">
+    <inertial>
+       <origin xyz="0 0 0" rpy="0 0 0"/>
+       <mass value="1e-5"/>
+       <inertia ixx="1e-6" ixy="0" ixz="0" iyy="1e-6" iyz="0" izz="1e-6"/>
+     </inertial>
+    <visual>
+      <origin xyz="0 0 0" rpy="0 0 0"/>
+      <geometry>
+        <mesh filename="package://my_robot/meshes/hokuyo.dae"/>
+      </geometry>
+    </visual>
+    <collision>
+      <origin xyz="0 0 0" rpy="0 0 0"/>
+      <geometry>
+        <box size="0.1 0.1 0.1"/>
+      </geometry>
+    </collision>
+  </link>
+  <joint type="fixed" name="hokuyo_joint">
+    <origin xyz="0.15 0 0.05" rpy="0 0 0"/>
+    <child link="hokuyo"/>
+    <parent link="chassis"/>
+    <axis xyz="0 1 0" rpy="0 0 0"/>
+    <limit effort="10000" velocity="1000"/>
+    <dynamics damping="1.0" friction="1.0"/>
+  </joint>
+  <joint name="camera_optical_joint" type="fixed">
+    <origin xyz="0 0 0" rpy="-1.5707 0 -1.5707"/>
+    <parent link="camera"/>
+    <child link="camera_optical"/>
+  </joint>
+  <link name="camera_optical">
+  </link>
 </robot>

Commit message: new: robot ready with teleop control
- add new world in gazebo

File: src/a1_bot/urdf/a1_bot.xacro (robot description, xacro)
@@ -1,4 +1,5 @@
 <?xml version='1.0'?>
 <robot name="a1_bot" xmlns:xacro="http://www.ros.org/wiki/xacro">
+  <xacro:include filename="$(find a1_bot)/urdf/a1_bot.gazebo" />
   <link name="robot_footprint"></link>
   <joint name="robot_footprint_joint" type="fixed">
@@ -142,5 +143,5 @@
   </link>
   <joint type="fixed" name="camera_joint">
-    <origin xyz="0.225 0 0" rpy="0 0 0"/>
+    <origin xyz="0.2 0 0" rpy="0 0 0"/>
     <child link="camera"/>
     <parent link="chassis"/>
@@ -158,5 +159,5 @@
       <origin xyz="0 0 0" rpy="0 0 0"/>
       <geometry>
-        <mesh filename="package://my_robot/meshes/hokuyo.dae"/>
+        <mesh filename="package://a1_bot/meshes/hokuyo.dae"/>
       </geometry>
     </visual>

Commit message: new: add sonar sensor to the robot

File: src/a1_bot/urdf/a1_bot.xacro (robot description, xacro)
@@ -1,8 +1,10 @@
 <?xml version='1.0'?>
-<robot name="a1_bot" xmlns:xacro="http://www.ros.org/wiki/xacro">
+<robot name="a1_bot"
+  xmlns:xacro="http://www.ros.org/wiki/xacro">
   <xacro:include filename="$(find a1_bot)/urdf/a1_bot.gazebo" />
   <link name="robot_footprint"></link>
   <joint name="robot_footprint_joint" type="fixed">
-    <origin xyz="0 0 0.124" rpy="0 0 0" /> <!-- keep robot wheels on the groud (offset value as per robot visual)-->
+    <origin xyz="0 0 0.124" rpy="0 0 0" />
+    <!-- keep robot wheels on the groud (offset value as per robot visual)-->
     <parent link="robot_footprint"/>
     <child link="chassis" />
@@ -13,9 +15,5 @@
       <mass value="15.0"/>
       <origin xyz="0.0 0 0" rpy=" 0 0 0"/>
-      <inertia
-          ixx="0.1" ixy="0" ixz="0"
-          iyy="0.1" iyz="0"
-          izz="0.1"
-      />
+      <inertia ixx="0.1" ixy="0" ixz="0" iyy="0.1" iyz="0" izz="0.1" />
     </inertial>
     <collision name='collision'>
@@ -57,21 +55,21 @@
   </link>
   <gazebo reference="chassis">
-     <material>Gazebo/Orange</material>
+    <material>Gazebo/Orange</material>
   </gazebo>
   <gazebo reference="left_wheel">
-     <material>Gazebo/Blue</material>
+    <material>Gazebo/Blue</material>
   </gazebo>
   <gazebo reference="right_wheel">
-     <material>Gazebo/Blue</material>
+    <material>Gazebo/Blue</material>
   </gazebo>
   <gazebo reference="camera">
-     <material>Gazebo/Red</material>
+    <material>Gazebo/Red</material>
   </gazebo>
   <link name="left_wheel">
     <inertial>
-       <origin xyz="0 0 0" rpy="0 1.5707 1.5707"/>
-       <mass value="5"/>
-       <inertia ixx="0.1" ixy="0" ixz="0" iyy="0.1" iyz="0" izz="0.1"/>
-     </inertial>
+      <origin xyz="0 0 0" rpy="0 1.5707 1.5707"/>
+      <mass value="5"/>
+      <inertia ixx="0.1" ixy="0" ixz="0" iyy="0.1" iyz="0" izz="0.1"/>
+    </inertial>
     <visual>
       <origin xyz="0 0 0" rpy="0 1.5707 1.5707"/>
@@ -97,8 +95,8 @@
   <link name="right_wheel">
     <inertial>
-       <origin xyz="0 0 0" rpy="0 1.5707 1.5707"/>
-       <mass value="5"/>
-       <inertia ixx="0.1" ixy="0" ixz="0" iyy="0.1" iyz="0" izz="0.1"/>
-     </inertial>
+      <origin xyz="0 0 0" rpy="0 1.5707 1.5707"/>
+      <mass value="5"/>
+      <inertia ixx="0.1" ixy="0" ixz="0" iyy="0.1" iyz="0" izz="0.1"/>
+    </inertial>
     <visual>
       <origin xyz="0 0 0" rpy="0 1.5707 1.5707"/>
@@ -122,11 +120,12 @@
     <dynamics damping="1.0" friction="1.0"/>
   </joint>
+  <!-- add 2D RGB camera sensor -->
   <link name="camera">
     <origin xyz="0 0 0" rpy="0 0 0"/>
     <inertial>
-       <origin xyz="0 0 0" rpy="0 0 0"/>
-       <mass value="0.1"/>
-       <inertia ixx="1e-6" ixy="0" ixz="0" iyy="1e-6" iyz="0" izz="1e-6"/>
-     </inertial>
+      <origin xyz="0 0 0" rpy="0 0 0"/>
+      <mass value="0.1"/>
+      <inertia ixx="1e-6" ixy="0" ixz="0" iyy="1e-6" iyz="0" izz="1e-6"/>
+    </inertial>
     <visual>
       <origin xyz="0 0 0" rpy="0 0 0"/>
@@ -150,10 +149,11 @@
     <dynamics damping="1.0" friction="1.0"/>
   </joint>
+  <!-- add laser range finder sensor -->
   <link name="hokuyo">
     <inertial>
-       <origin xyz="0 0 0" rpy="0 0 0"/>
-       <mass value="1e-5"/>
-       <inertia ixx="1e-6" ixy="0" ixz="0" iyy="1e-6" iyz="0" izz="1e-6"/>
-     </inertial>
+      <origin xyz="0 0 0" rpy="0 0 0"/>
+      <mass value="1e-5"/>
+      <inertia ixx="1e-6" ixy="0" ixz="0" iyy="1e-6" iyz="0" izz="1e-6"/>
+    </inertial>
     <visual>
       <origin xyz="0 0 0" rpy="0 0 0"/>
@@ -184,3 +184,29 @@
   <link name="camera_optical">
   </link>
+  <!-- add sonar sensor to robot -->
+  <link name="base_sonar">
+    <collision>
+      <origin xyz="0 0 0" rpy="0 0 0"/>
+      <geometry>
+        <box size="0.01 0.01 0.01"/>
+      </geometry>
+    </collision>
+    <visual>
+      <origin xyz="0 0 0" rpy="0 0 0"/>
+      <geometry>
+        <box size="0.01 0.01 0.01"/>
+      </geometry>
+    </visual>
+    <inertial>
+      <mass value="1e-5" />
+      <origin xyz="0 0 0" rpy="0 0 0"/>
+      <inertia ixx="1e-6" ixy="0" ixz="0" iyy="1e-6" iyz="0" izz="1e-6" />
+    </inertial>
+  </link>
+  <joint name="sonar_joint" type="fixed">
+    <axis xyz="0 1 0" />
+    <origin rpy="0 1.57 0" xyz="0.15 -0.1 -0.03" />
+    <parent link="chassis"/>
+    <child link="base_sonar"/>
+  </joint>
 </robot>
